File: pcb/heli/radio.kicad_sch (KiCad schematic)
At the start: 16 parts

Commit message: 
Parts:
- C16, C17, C18, C19, C20, C21, C22, C23, C24: renamed from C?; footprint (none) -> Capacitor_SMD:C_0603_1608Metric
- L1, L2, L3: renamed from L?; footprint (none) -> Inductor_SMD:L_0603_1608Metric
- R3, R6: renamed from R?; footprint (none) -> Resistor_SMD:R_0603_1608Metric
- Y2: renamed from Y?; footprint (none) -> Crystal:Crystal_HC49-4H_Vertical
- gave numbers to parts that had none: 1
Connections:
- net at U5.13 (ANT2): now also L1.2, L3.1

Commit message: 
Parts:
- Y2: footprint Crystal:Crystal_HC49-4H_Vertical -> Crystal:Crystal_SMD_HC49-SD
Changed lines of the file:
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@@
     (property "Reference" "Y2" (id 0) (at 147.32 69.9348 0))
     (property "Value" "16MHz" (id 1) (at 147.32 72.4717 0))
-    (property "Footprint" "Crystal:Crystal_HC49-4H_Vertical" (id 2) (at 147.32 76.2 0)
+    (property "Footprint" "Crystal:Crystal_SMD_HC49-SD" (id 2) (at 147.32 76.2 0)
       (effects (font (size 1.27 1.27)) hide)
     )

Commit message: 
Parts:
- added AE1: Antenna_Shield, sparkfun:TRACE_ANTENNA_2.4GHZ_15.2MM, symbol Device:Antenna_Shield
Connections:
- net 50ohm: now also AE1.1 (A)
- net GND: now also AE1.2 (Shield)
Changed lines of the file:
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@@
     (pin "1")
+  )
+  (symbol (lib_id "Device:Antenna_Shield") (at 182.88 58.42 0) (unit 1)
+    (in_bom yes) (on_board yes) (fields_autoplaced)
+    (property "Reference" "AE1" (id 0) (at 186.055 56.9503 0)
+      (effects (font (size 1.27 1.27)) (justify left))
+    )
+    (property "Value" "Antenna_Shield" (id 1) (at 186.055 59.4872 0)
+      (effects (font (size 1.27 1.27)) (justify left))
+    )
+    (property "Footprint" "sparkfun:TRACE_ANTENNA_2.4GHZ_15.2MM" (id 2) (at 182.88 55.88 0)
+      (effects (font (size 1.27 1.27)) hide)
+    )
+    (property "Datasheet" "~" (id 3) (at 182.88 55.88 0)
+      (effects (font (size 1.27 1.27)) hide)
+    )
+    (pin "1")
+    (pin "2")
   )
   (symbol (lib_id "Device:R") (at 92.71 71.12 90) (unit 1)
@@
     (pin "2")
   )
+  (symbol (lib_id "power:GND") (at 185.42 63.5 0) (unit 1)
+    (in_bom yes) (on_board yes) (fields_autoplaced)
+    (property "Reference" "#PWR031" (id 0) (at 185.42 69.85 0)
+      (effects (font (size 1.27 1.27)) hide)
+    )
+    (property "Value" "GND" (id 1) (at 185.42 67.9434 0))
+    (property "Footprint" "" (id 2) (at 185.42 63.5 0)
+      (effects (font (size 1.27 1.27)) hide)
+    )
+    (property "Datasheet" "" (id 3) (at 185.42 63.5 0)
+      (effects (font (size 1.27 1.27)) hide)
+    )
+    (pin "1")
+  )
   (symbol (lib_id "power:GND") (at 140.97 43.18 180) (unit 1)

Commit message: 
Parts:
- C17, C20: value 22pF -> 30pF
Changed lines of the file:
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@@
       (effects (font (size 1.27 1.27)) (justify left))
     )
-    (property "Value" "22pF" (id 1) (at 136.779 90.6022 0)
+    (property "Value" "30pF" (id 1) (at 136.779 90.6022 0)
       (effects (font (size 1.27 1.27)) (justify left))
     )
@@
       (effects (font (size 1.27 1.27)) (justify left))
     )
-    (property "Value" "22pF" (id 1) (at 160.401 90.0942 0)
+    (property "Value" "30pF" (id 1) (at 160.401 90.0942 0)
       (effects (font (size 1.27 1.27)) (justify left))
     )

Commit message: 
Parts:
- U5: DIGIKEY (none) -> https://www.digikey.de/en/products/detail/nordic-semiconduc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
- Y2: DIGIKEY (none) -> https://www.digikey.de/en/products/detail/ecs-inc/ECS-160-2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
Changed lines of the file:
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@@
+      (effects (font (size 1.27 1.27)) hide)
+    )
+    (property "DIGIKEY" "https://www.digikey.de/en/products/detail/nordic-semiconductor-asa/NRF24L01P-T/4626383" (id 4) (at 111.76 63.5 0)
       (effects (font (size 1.27 1.27)) hide)
     )
@@
       (effects (font (size 1.27 1.27)) hide)
     )
+    (property "DIGIKEY" "https://www.digikey.de/en/products/detail/ecs-inc/ECS-160-20-3X-EN-TR/2676623" (id 4) (at 147.32 76.2 0)
+      (effects (font (size 1.27 1.27)) hide)
+    )

Commit message: 
Parts:
- AE1: now left out of the parts list
- R6: DIGIKEY (none) -> https://www.digikey.de/en/products/detail/walsin-technology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
Changed lines of the file:
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@@
   )
   (symbol (lib_id "Device:Antenna_Shield") (at 182.88 58.42 0) (unit 1)
-    (in_bom yes) (on_board yes) (fields_autoplaced)
+    (in_bom no) (on_board yes) (fields_autoplaced)
     (property "Reference" "AE1" (id 0) (at 186.055 56.9503 0)
       (effects (font (size 1.27 1.27)) (justify left))
@@
       (effects (font (size 1.27 1.27)) hide)
     )
+    (property "DIGIKEY" "https://www.digikey.de/en/products/detail/walsin-technology-corporation/WR06X1004FTL/13241115" (id 4) (at 147.32 82.804 0)
+      (effects (font (size 1.27 1.27)) hide)
+    )

Commit message: 
Parts:
- R6: DIGIKEY https://www.digikey.de/en/products/detail/walsin-technology-corporation/WR06X1004FTL/13241115 -> https://www.digikey.de/en/products/detail/walsin-technology-corporation/WR06X105-JTL/13239221
Changed lines of the file:
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@@
       (effects (font (size 1.27 1.27)) hide)
     )
-    (property "DIGIKEY" "https://www.digikey.de/en/products/detail/walsin-technology-corporation/WR06X1004FTL/13241115" (id 4) (at 147.32 82.804 0)
+    (property "DIGIKEY" "https://www.digikey.de/en/products/detail/walsin-technology-corporation/WR06X105-JTL/13239221" (id 4) (at 147.32 82.804 0)
       (effects (font (size 1.27 1.27)) hide)
     )

Commit message: 
Parts:
- AE1: DIGIKEY (none) -> -
- C16, C23, C24: DIGIKEY (none) -> https://www.digikey.de/en/products/detail/w%C3%BCrth-elektr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
- C17, C20: DIGIKEY (none) -> https://www.digikey.de/en/products/detail/stackpole-electro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
- C18: footprint Capacitor_SMD:C_0603_1608Metric -> Capacitor_SMD:C_0402_1005Metric; DIGIKEY (none) -> https://www.digikey.de/en/products/detail/w%C3%BCrth-elektr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
- C19: footprint Capacitor_SMD:C_0603_1608Metric -> Capacitor_SMD:C_0402_1005Metric; DIGIKEY (none) -> https://www.digikey.de/en/products/detail/yageo/CC0402CRNPO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
- C21, C22: footprint Capacitor_SMD:C_0603_1608Metric -> Capacitor_SMD:C_0402_1005Metric; DIGIKEY (none) -> https://www.digikey.de/en/products/detail/yageo/CC0402BRNPO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
- L1, L2, L3: footprint Inductor_SMD:L_0603_1608Metric -> Inductor_SMD:L_0402_1005Metric; DIGIKEY (none) -> https://www.digikey.de/en/products/detail/w%C3%BCrth-elektr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
- R3: DIGIKEY (none) -> https://www.digikey.de/en/products/detail/walsin-technology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
Changed lines of the file:
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@@
+      (effects (font (size 1.27 1.27)) hide)
+    )
+    (property "DIGIKEY" "https://www.digikey.de/en/products/detail/w%C3%BCrth-elektronik/885012206092/5453865" (id 4) (at 91.948 82.55 0)
       (effects (font (size 1.27 1.27)) hide)
     )
@@
       (effects (font (size 1.27 1.27)) (justify left))
     )
-    (property "Footprint" "Capacitor_SMD:C_0603_1608Metric" (id 2) (at 141.9352 50.8 0)
+    (property "Footprint" "Capacitor_SMD:C_0402_1005Metric" (id 2) (at 141.9352 50.8 0)
       (effects (font (size 1.27 1.27)) hide)
     )
     (property "Datasheet" "~" (id 3) (at 140.97 46.99 0)
+      (effects (font (size 1.27 1.27)) hide)
+    )
+    (property "DIGIKEY" "https://www.digikey.de/en/products/detail/w%C3%BCrth-elektronik/885012205008/5453358" (id 4) (at 140.97 46.99 0)
       (effects (font (size 1.27 1.27)) hide)
     )
@@
     )
     (property "Datasheet" "~" (id 3) (at 182.88 55.88 0)
+      (effects (font (size 1.27 1.27)) hide)
+    )
+    (property "DIGIKEY" "-" (id 4) (at 182.88 58.42 0)
       (effects (font (size 1.27 1.27)) hide)
     )
@@
       (effects (font (size 1.27 1.27)) hide)
     )
+    (property "DIGIKEY" "https://www.digikey.de/en/products/detail/walsin-technology-corporation/WR06X2202FTL/13239195" (id 4) (at 92.71 71.12 0)
+      (effects (font (size 1.27 1.27)) hide)
+    )
     (pin "1")
     (pin "2")
@@
     )
     (property "Datasheet" "~" (id 3) (at 133.858 88.9 0)
+      (effects (font (size 1.27 1.27)) hide)
+    )
+    (property "DIGIKEY" "https://www.digikey.de/en/products/detail/stackpole-electronics-inc/CML0603C0G300JT50V/10659967" (id 4) (at 133.858 88.9 0)
       (effects (font (size 1.27 1.27)) hide)
     )
@@
     (property "Reference" "L3" (id 0) (at 151.13 59.2922 90))
     (property "Value" "3.9nH" (id 1) (at 151.13 61.8291 90))
-    (property "Footprint" "Inductor_SMD:L_0603_1608Metric" (id 2) (at 151.13 63.5 0)
+    (property "Footprint" "Inductor_SMD:L_0402_1005Metric" (id 2) (at 151.13 63.5 0)
       (effects (font (size 1.27 1.27)) hide)
     )
     (property "Datasheet" "~" (id 3) (at 151.13 63.5 0)
+      (effects (font (size 1.27 1.27)) hide)
+    )
+    (property "DIGIKEY" "https://www.digikey.de/en/products/detail/w%C3%BCrth-elektronik/7447840039G/14670181" (id 4) (at 151.13 63.5 0)
       (effects (font (size 1.27 1.27)) hide)
     )
@@
     (property "Reference" "C21" (id 0) (at 163.83 57.6412 90))
     (property "Value" "1.5pF" (id 1) (at 163.83 60.1781 90))
-    (property "Footprint" "Capacitor_SMD:C_0603_1608Metric" (id 2) (at 167.64 62.5348 0)
+    (property "Footprint" "Capacitor_SMD:C_0402_1005Metric" (id 2) (at 167.64 62.5348 0)
       (effects (font (size 1.27 1.27)) hide)
     )
     (property "Datasheet" "~" (id 3) (at 163.83 63.5 0)
+      (effects (font (size 1.27 1.27)) hide)
+    )
+    (property "DIGIKEY" "https://www.digikey.de/en/products/detail/yageo/CC0402BRNPO9BN1R5/5883186" (id 4) (at 163.83 63.5 0)
       (effects (font (size 1.27 1.27)) hide)
     )
@@
       (effects (font (size 1.27 1.27)) hide)
     )
+    (property "DIGIKEY" "https://www.digikey.de/en/products/detail/w%C3%BCrth-elektronik/885012206014/5453788" (id 4) (at 194.31 46.99 0)
+      (effects (font (size 1.27 1.27)) hide)
+    )
     (pin "1")
     (pin "2")
@@
       (effects (font (size 1.27 1.27)) (justify right))
     )
-    (property "Footprint" "Capacitor_SMD:C_0603_1608Metric" (id 2) (at 169.2148 66.04 0)
+    (property "Footprint" "Capacitor_SMD:C_0402_1005Metric" (id 2) (at 169.2148 66.04 0)
       (effects (font (size 1.27 1.27)) hide)
     )
     (property "Datasheet" "~" (id 3) (at 170.18 69.85 0)
+      (effects (font (size 1.27 1.27)) hide)
+    )
+    (property "DIGIKEY" "https://www.digikey.de/en/products/detail/yageo/CC0402BRNPO9BN1R0/5883183" (id 4) (at 170.18 69.85 0)
       (effects (font (size 1.27 1.27)) hide)
     )
@@
       (effects (font (size 1.27 1.27)) (justify left))
     )
-    (property "Footprint" "Capacitor_SMD:C_0603_1608Metric" (id 2) (at 154.6352 50.8 0)
+    (property "Footprint" "Capacitor_SMD:C_0402_1005Metric" (id 2) (at 154.6352 50.8 0)
       (effects (font (size 1.27 1.27)) hide)
     )
@@
       (effects (font (size 1.27 1.27)) hide)
     )
+    (property "DIGIKEY" "https://www.digikey.de/en/products/detail/yageo/CC0402CRNPO9BN4R7/2103105" (id 4) (at 153.67 46.99 0)
+      (effects (font (size 1.27 1.27)) hide)
+    )
     (pin "1")
     (pin "2")
@@
     )
     (property "Datasheet" "~" (id 3) (at 157.48 88.392 0)
+      (effects (font (size 1.27 1.27)) hide)
+    )
+    (property "DIGIKEY" "https://www.digikey.de/en/products/detail/stackpole-electronics-inc/CML0603C0G300JT50V/10659967" (id 4) (at 157.48 88.392 0)
       (effects (font (size 1.27 1.27)) hide)
     )
@@
       (effects (font (size 1.27 1.27)) (justify left))
     )
-    (property "Footprint" "Inductor_SMD:L_0603_1608Metric" (id 2) (at 135.89 59.69 0)
+    (property "Footprint" "Inductor_SMD:L_0402_1005Metric" (id 2) (at 135.89 59.69 0)
       (effects (font (size 1.27 1.27)) hide)
     )
     (property "Datasheet" "~" (id 3) (at 135.89 59.69 0)
+      (effects (font (size 1.27 1.27)) hide)
+    )
+    (property "DIGIKEY" "https://www.digikey.de/en/products/detail/w%C3%BCrth-elektronik/7847803820/14640462" (id 4) (at 135.89 59.69 0)
       (effects (font (size 1.27 1.27)) hide)
     )
@@
     (property "Reference" "L2" (id 0) (at 151.13 51.6722 90))
     (property "Value" "2.7nH" (id 1) (at 151.13 54.2091 90))
-    (property "Footprint" "Inductor_SMD:L_0603_1608Metric" (id 2) (at 151.13 55.88 0)
+    (property "Footprint" "Inductor_SMD:L_0402_1005Metric" (id 2) (at 151.13 55.88 0)
       (effects (font (size 1.27 1.27)) hide)
     )
@@
       (effects (font (size 1.27 1.27)) hide)
     )
+    (property "DIGIKEY" "https://www.digikey.de/en/products/detail/w%C3%BCrth-elektronik/7447840027G/14670139" (id 4) (at 151.13 55.88 0)
+      (effects (font (size 1.27 1.27)) hide)
+    )
     (pin "1")
     (pin "2")
@@
       (effects (font (size 1.27 1.27)) hide)
     )
+    (property "DIGIKEY" "https://www.digikey.de/en/products/detail/w%C3%BCrth-elektronik/885012206083/5453856" (id 4) (at 204.47 46.99 0)
+      (effects (font (size 1.27 1.27)) hide)
+    )
