File: pcb/heli/radio.kicad_sch (KiCad schematic)
At the start: 17 parts, among them U5 NRF24L01, Y2 16MHz

Commit message: 
Parts:
- C16: DIGIKEY https://www.digikey.de/en/products/detail/w%C3%BCrth-elektr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 -> 732-8010-1-ND
- C17, C20: DIGIKEY https://www.digikey.de/en/products/detail/stackpole-electro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 -> 738-CML0603C0G300JT50VCT-ND
- C18: DIGIKEY https://www.digikey.de/en/products/detail/w%C3%BCrth-elektr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 -> 732-7503-1-ND
- C19: DIGIKEY https://www.digikey.de/en/products/detail/yageo/CC0402CRNPO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 -> 311-1367-1-ND
- C21: DIGIKEY https://www.digikey.de/en/products/detail/yageo/CC0402BRNPO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 -> 311-3323-1-ND
- C22: DIGIKEY https://www.digikey.de/en/products/detail/yageo/CC0402BRNPO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 -> 311-3613-1-ND
- C23: DIGIKEY https://www.digikey.de/en/products/detail/w%C3%BCrth-elektr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 -> 732-7933-1-ND
- C24: DIGIKEY https://www.digikey.de/en/products/detail/w%C3%BCrth-elektr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 -> 732-8001-1-ND
- L1: DIGIKEY https://www.digikey.de/en/products/detail/w%C3%BCrth-elektr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 -> 732-7847803820CT-ND
- L2: DIGIKEY https://www.digikey.de/en/products/detail/w%C3%BCrth-elektr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 -> 732-7447840027GCT-ND
- L3: DIGIKEY https://www.digikey.de/en/products/detail/w%C3%BCrth-elektr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 -> 732-7447840039GCT-ND
- R3: DIGIKEY https://www.digikey.de/en/products/detail/walsin-technology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 -> 1292-WR06X2202FTLCT-ND
- R6: DIGIKEY https://www.digikey.de/en/products/detail/walsin-technology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 -> 1292-WR06X105JTLCT-ND
- U5: DIGIKEY https://www.digikey.de/en/products/detail/nordic-semiconduc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 -> 1490-1019-ND
- Y2: DIGIKEY https://www.digikey.de/en/products/detail/ecs-inc/ECS-160-2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 -> XC1793CT-ND
Changed lines of the file:
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@@
       (effects (font (size 1.27 1.27)) hide)
     )
-    (property "DIGIKEY" "https://www.digikey.de/en/products/detail/nordic-semiconductor-asa/NRF24L01P-T/4626383" (id 4) (at 111.76 63.5 0)
+    (property "DIGIKEY" "1490-1019-ND" (id 4) (at 111.76 63.5 0)
       (effects (font (size 1.27 1.27)) hide)
     )
@@
       (effects (font (size 1.27 1.27)) hide)
     )
-    (property "DIGIKEY" "https://www.digikey.de/en/products/detail/w%C3%BCrth-elektronik/885012206092/5453865" (id 4) (at 91.948 82.55 0)
+    (property "DIGIKEY" "732-8010-1-ND" (id 4) (at 91.948 82.55 0)
       (effects (font (size 1.27 1.27)) hide)
     )
@@
       (effects (font (size 1.27 1.27)) hide)
     )
-    (property "DIGIKEY" "https://www.digikey.de/en/products/detail/ecs-inc/ECS-160-20-3X-EN-TR/2676623" (id 4) (at 147.32 76.2 0)
+    (property "DIGIKEY" "XC1793CT-ND" (id 4) (at 147.32 76.2 0)
       (effects (font (size 1.27 1.27)) hide)
     )
@@
       (effects (font (size 1.27 1.27)) hide)
     )
-    (property "DIGIKEY" "https://www.digikey.de/en/products/detail/w%C3%BCrth-elektronik/885012205008/5453358" (id 4) (at 140.97 46.99 0)
+    (property "DIGIKEY" "732-7503-1-ND" (id 4) (at 140.97 46.99 0)
       (effects (font (size 1.27 1.27)) hide)
     )
@@
       (effects (font (size 1.27 1.27)) hide)
     )
-    (property "DIGIKEY" "https://www.digikey.de/en/products/detail/walsin-technology-corporation/WR06X2202FTL/13239195" (id 4) (at 92.71 71.12 0)
+    (property "DIGIKEY" "1292-WR06X2202FTLCT-ND" (id 4) (at 92.71 71.12 0)
       (effects (font (size 1.27 1.27)) hide)
     )
@@
       (effects (font (size 1.27 1.27)) hide)
     )
-    (property "DIGIKEY" "https://www.digikey.de/en/products/detail/stackpole-electronics-inc/CML0603C0G300JT50V/10659967" (id 4) (at 133.858 88.9 0)
+    (property "DIGIKEY" "738-CML0603C0G300JT50VCT-ND" (id 4) (at 133.858 88.9 0)
       (effects (font (size 1.27 1.27)) hide)
     )
@@
       (effects (font (size 1.27 1.27)) hide)
     )
-    (property "DIGIKEY" "https://www.digikey.de/en/products/detail/w%C3%BCrth-elektronik/7447840039G/14670181" (id 4) (at 151.13 63.5 0)
+    (property "DIGIKEY" "732-7447840039GCT-ND" (id 4) (at 151.13 63.5 0)
       (effects (font (size 1.27 1.27)) hide)
     )
@@
       (effects (font (size 1.27 1.27)) hide)
     )
-    (property "DIGIKEY" "https://www.digikey.de/en/products/detail/walsin-technology-corporation/WR06X105-JTL/13239221" (id 4) (at 147.32 82.804 0)
+    (property "DIGIKEY" "1292-WR06X105JTLCT-ND" (id 4) (at 147.32 82.804 0)
       (effects (font (size 1.27 1.27)) hide)
     )
@@
       (effects (font (size 1.27 1.27)) hide)
     )
-    (property "DIGIKEY" "https://www.digikey.de/en/products/detail/yageo/CC0402BRNPO9BN1R5/5883186" (id 4) (at 163.83 63.5 0)
+    (property "DIGIKEY" "311-3323-1-ND" (id 4) (at 163.83 63.5 0)
       (effects (font (size 1.27 1.27)) hide)
     )
@@
       (effects (font (size 1.27 1.27)) hide)
     )
-    (property "DIGIKEY" "https://www.digikey.de/en/products/detail/w%C3%BCrth-elektronik/885012206014/5453788" (id 4) (at 194.31 46.99 0)
+    (property "DIGIKEY" "732-7933-1-ND" (id 4) (at 194.31 46.99 0)
       (effects (font (size 1.27 1.27)) hide)
     )
@@
       (effects (font (size 1.27 1.27)) hide)
     )
-    (property "DIGIKEY" "https://www.digikey.de/en/products/detail/yageo/CC0402BRNPO9BN1R0/5883183" (id 4) (at 170.18 69.85 0)
+    (property "DIGIKEY" "311-3613-1-ND" (id 4) (at 170.18 69.85 0)
       (effects (font (size 1.27 1.27)) hide)
     )
@@
       (effects (font (size 1.27 1.27)) hide)
     )
-    (property "DIGIKEY" "https://www.digikey.de/en/products/detail/yageo/CC0402CRNPO9BN4R7/2103105" (id 4) (at 153.67 46.99 0)
+    (property "DIGIKEY" "311-1367-1-ND" (id 4) (at 153.67 46.99 0)
       (effects (font (size 1.27 1.27)) hide)
     )
@@
       (effects (font (size 1.27 1.27)) hide)
     )
-    (property "DIGIKEY" "https://www.digikey.de/en/products/detail/stackpole-electronics-inc/CML0603C0G300JT50V/10659967" (id 4) (at 157.48 88.392 0)
+    (property "DIGIKEY" "738-CML0603C0G300JT50VCT-ND" (id 4) (at 157.48 88.392 0)
       (effects (font (size 1.27 1.27)) hide)
     )
@@
       (effects (font (size 1.27 1.27)) hide)
     )
-    (property "DIGIKEY" "https://www.digikey.de/en/products/detail/w%C3%BCrth-elektronik/7847803820/14640462" (id 4) (at 135.89 59.69 0)
+    (property "DIGIKEY" "732-7847803820CT-ND" (id 4) (at 135.89 59.69 0)
       (effects (font (size 1.27 1.27)) hide)
     )
@@
       (effects (font (size 1.27 1.27)) hide)
     )
-    (property "DIGIKEY" "https://www.digikey.de/en/products/detail/w%C3%BCrth-elektronik/7447840027G/14670139" (id 4) (at 151.13 55.88 0)
+    (property "DIGIKEY" "732-7447840027GCT-ND" (id 4) (at 151.13 55.88 0)
       (effects (font (size 1.27 1.27)) hide)
     )
@@
       (effects (font (size 1.27 1.27)) hide)
     )
-    (property "DIGIKEY" "https://www.digikey.de/en/products/detail/w%C3%BCrth-elektronik/885012206083/5453856" (id 4) (at 204.47 46.99 0)
-      (effects (font (size 1.27 1.27)) hide)
-    )
+    (property "DIGIKEY" "732-8001-1-ND" (id 4) (at 204.47 46.99 0)
+      (effects (font (size 1.27 1.27)) hide)
+    )

Commit message: 
Parts:
- added C29: 100nF, Capacitor_SMD:C_0603_1608Metric, symbol Device:C
Connections:
- net 3.3V: now also C29.1
- net GND: now also C29.2
Changed lines of the file:
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@@
+    )
+  )
+  (global_label "3.3V" (shape input) (at 214.63 43.18 90) (fields_autoplaced)
+    (effects (font (size 1.27 1.27)) (justify left))
+    (property "Intersheet References" "${INTERSHEET_REFS}" (id 0) (at 214.5506 36.6545 90)
+      (effects (font (size 1.27 1.27)) (justify left) hide)
     )
   )
@@
     )
     (pin "1")
+  )
+  (symbol (lib_id "Device:C") (at 214.63 46.99 0) (unit 1)
+    (in_bom yes) (on_board yes) (fields_autoplaced)
+    (property "Reference" "C29" (id 0) (at 217.551 46.1553 0)
+      (effects (font (size 1.27 1.27)) (justify left))
+    )
+    (property "Value" "100nF" (id 1) (at 217.551 48.6922 0)
+      (effects (font (size 1.27 1.27)) (justify left))
+    )
+    (property "Footprint" "Capacitor_SMD:C_0603_1608Metric" (id 2) (at 215.5952 50.8 0)
+      (effects (font (size 1.27 1.27)) hide)
+    )
+    (property "Datasheet" "~" (id 3) (at 214.63 46.99 0)
+      (effects (font (size 1.27 1.27)) hide)
+    )
+    (property "DIGIKEY" "1276-1935-1-ND" (id 4) (at 214.63 46.99 0)
+      (effects (font (size 1.27 1.27)) hide)
+    )
+    (pin "1")
+    (pin "2")
   )
   (symbol (lib_id "power:GND") (at 116.84 83.82 0) (unit 1)
@@
       (effects (font (size 1.27 1.27)) hide)
     )
+    (pin "1")
+  )
+  (symbol (lib_id "power:GND") (at 214.63 50.8 0) (unit 1)
+    (in_bom yes) (on_board yes) (fields_autoplaced)
+    (property "Reference" "#PWR033" (id 0) (at 214.63 57.15 0)
+      (effects (font (size 1.27 1.27)) hide)
+    )
+    (property "Value" "GND" (id 1) (at 214.63 55.2434 0))
+    (property "Footprint" "" (id 2) (at 214.63 50.8 0)
+      (effects (font (size 1.27 1.27)) hide)
+    )
+    (property "Datasheet" "" (id 3) (at 214.63 50.8 0)
+      (effects (font (size 1.27 1.27)) hide)
+    )

Commit message: 
Connections:
- net 50ohm renamed RADIO50ohm
Changed lines of the file:
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@@
     (stroke (width 0) (type default) (color 0 0 0 0))
   )
-  (label "50ohm" (at 182.88 63.5 180)
+  (label "RADIO50ohm" (at 182.88 63.5 180)
     (effects (font (size 1.27 1.27)) (justify right bottom))
   )
