File: pcb/heli/heli.kicad_sch (KiCad schematic)
At the start: 32 parts, among them J1 Batterie, J2 Debug, J4 Servo, J5 Servo, Q1 IRLZ44N, SW1 SW_MEC_5E, U1 AZ1117-3.3, U2 MPU-6050, U3 STM32F103CBTx, Y1 8MHz

Commit message: 
Parts:
- D1: DIGIKEY (none) -> https://www.digikey.de/en/products/detail/liteon/LTST-C190K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
- R14: DIGIKEY (none) -> https://www.digikey.de/en/products/detail/walsin-technology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
Connections:
- net GPS_NRST: now reaches U3.14 (PA4)
Other:
- sheet GPS ports: added RESET; removed none
Changed lines of the file:
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@@
+    (stroke (width 0) (type default) (color 0 0 0 0))
+  )
+  (wire (pts (xy 198.755 137.16) (xy 198.755 137.795))
     (stroke (width 0) (type default) (color 0 0 0 0))
   )
@@
     )
   )
+  (global_label "GPS_NRST" (shape input) (at 198.755 137.16 90) (fields_autoplaced)
+    (effects (font (size 1.27 1.27)) (justify left))
+    (property "Intersheet References" "${INTERSHEET_REFS}" (id 0) (at 198.6756 125.2521 90)
+      (effects (font (size 1.27 1.27)) (justify left) hide)
+    )
+  )
   (global_label "RESET" (shape input) (at 247.65 32.385 180) (fields_autoplaced)
     (effects (font (size 1.27 1.27)) (justify right))
@@
     (property "Intersheet References" "${INTERSHEET_REFS}" (id 0) (at 178.8038 147.8756 0)
       (effects (font (size 1.27 1.27)) (justify right) hide)
+    )
+  )
+  (global_label "GPS_NRST" (shape output) (at 169.545 77.47 0) (fields_autoplaced)
+    (effects (font (size 1.27 1.27)) (justify left))
+    (property "Intersheet References" "${INTERSHEET_REFS}" (id 0) (at 181.4529 77.3906 0)
+      (effects (font (size 1.27 1.27)) (justify left) hide)
     )
   )
@@
     )
     (property "Datasheet" "~" (id 3) (at 79.375 78.74 0)
+      (effects (font (size 1.27 1.27)) hide)
+    )
+    (property "DIGIKEY" "https://www.digikey.de/en/products/detail/walsin-technology-corporation/WR06X1004FTL/13241115" (id 4) (at 79.375 78.74 0)
       (effects (font (size 1.27 1.27)) hide)
     )
@@
       (effects (font (size 1.27 1.27)) hide)
     )
+    (property "DIGIKEY" "https://www.digikey.de/en/products/detail/liteon/LTST-C190KRKT/386817" (id 4) (at 109.22 22.225 0)
+      (effects (font (size 1.27 1.27)) hide)
+    )
     (pin "1")
     (pin "2")
@@
     (pin "CSN" input (at 189.865 151.13 180)
       (effects (font (size 1.27 1.27)) (justify left))
+    )
+    (pin "RESET" input (at 198.755 137.795 90)
+      (effects (font (size 1.27 1.27)) (justify right))
     )
   )
@@
       (reference "#PWR0118") (unit 1) (value "GND") (footprint "")
     )
+    (path "/ff163e09-1c9a-4e9f-9fc2-cd2f8ec1c6f1/70e8289e-2779-4378-af50-a144d25bf420"
+      (reference "#PWR0119") (unit 1) (value "GND") (footprint "")
+    )
     (path "/8972c389-56a6-466a-9271-66b0ec918c0e/513d8dee-6e00-4610-92f7-bea566c6ff2b"
       (reference "AE1") (unit 1) (value "Antenna_Shield") (footprint "sparkfun:TRACE_ANTENNA_2.4GHZ_15.2MM")
@@
       (reference "C26") (unit 1) (value "100nF") (footprint "Capacitor_SMD:C_0603_1608Metric")
     )
+    (path "/ff163e09-1c9a-4e9f-9fc2-cd2f8ec1c6f1/d402a1a9-68bf-4d32-ae32-c37e50644652"
+      (reference "C27") (unit 1) (value "100nF") (footprint "Capacitor_SMD:C_0603_1608Metric")
+    )
     (path "/b28a0e5f-aecf-489c-9fc5-7ef0cd88e703"
       (reference "D1") (unit 1) (value "LED") (footprint "LED_SMD:LED_0603_1608Metric")
@@
       (reference "R14") (unit 1) (value "1M") (footprint "Resistor_SMD:R_0603_1608Metric")
     )
+    (path "/ff163e09-1c9a-4e9f-9fc2-cd2f8ec1c6f1/be937376-49ab-49c3-a6e4-e63ccde3693d"
+      (reference "R15") (unit 1) (value "10k") (footprint "Resistor_SMD:R_0603_1608Metric")
+    )
     (path "/adfea837-fd00-47ad-b3eb-1946872908eb"

Commit message: 
Parts:
- R14: DIGIKEY https://www.digikey.de/en/products/detail/walsin-technology-corporation/WR06X1004FTL/13241115 -> https://www.digikey.de/en/products/detail/walsin-technology-corporation/WR06X105-JTL/13239221
Changed lines of the file:
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@@
       (effects (font (size 1.27 1.27)) hide)
     )
-    (property "DIGIKEY" "https://www.digikey.de/en/products/detail/walsin-technology-corporation/WR06X1004FTL/13241115" (id 4) (at 79.375 78.74 0)
+    (property "DIGIKEY" "https://www.digikey.de/en/products/detail/walsin-technology-corporation/WR06X105-JTL/13239221" (id 4) (at 79.375 78.74 0)
       (effects (font (size 1.27 1.27)) hide)
     )

Commit message: 
Parts:
- C1, C3, Q1, U1: DIGIKEY (none) -> -
- C10, C11, C12, C13, C15, C9: DIGIKEY (none) -> https://www.digikey.de/en/products/detail/samsung-electro-m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
- C14: footprint Capacitor_SMD:C_0603_1608Metric -> Capacitor_SMD:CP_Elec_5x5.9; DIGIKEY (none) -> -
- C2, C8: DIGIKEY (none) -> https://www.digikey.de/en/products/detail/w%C3%BCrth-elektr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
- C4, C5: value 0.1uF -> 100nF; DIGIKEY (none) -> https://www.digikey.de/en/products/detail/samsung-electro-m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
- C6, C7: DIGIKEY (none) -> https://www.digikey.de/en/products/detail/stackpole-electro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
- R1, R2, R5, R7: DIGIKEY (none) -> https://www.digikey.de/en/products/detail/walsin-technology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
- R4: DIGIKEY (none) -> https://www.digikey.de/en/products/detail/yageo/RC0603FR-07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

Commit message: 
Parts:
- C1, C3: footprint Capacitor_SMD:CP_Elec_4x5.4 -> Capacitor_SMD:CP_Elec_5x5.4
- C10, C11, C12, C13, C15, C4, C5, C9: DIGIKEY https://www.digikey.de/en/products/detail/samsung-electro-m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 -> 1276-1935-1-ND
- C2: DIGIKEY https://www.digikey.de/en/products/detail/w%C3%BCrth-elektr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 -> 732-7933-1-ND
- C6, C7: DIGIKEY https://www.digikey.de/en/products/detail/stackpole-electro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 -> 738-CML0603C0G300JT50VCT-ND
- C8: DIGIKEY https://www.digikey.de/en/products/detail/w%C3%BCrth-elektr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 -> 732-8003-1-ND
- D1: DIGIKEY https://www.digikey.de/en/products/detail/liteon/LTST-C190K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 -> 160-1436-1-ND
- J1, J2, J4, J5: DIGIKEY https://www.digikey.de/en/products/detail/adam-tech/PH1-10-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 -> 2057-PH1-10-UA-ND
- R1, R2, R5, R7: DIGIKEY https://www.digikey.de/en/products/detail/walsin-technology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 -> 1292-WR06X103JTLCT-ND
- R14: DIGIKEY https://www.digikey.de/en/products/detail/walsin-technology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 -> 1292-WR06X105JTLCT-ND
- R4: DIGIKEY https://www.digikey.de/en/products/detail/yageo/RC0603FR-07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 -> 311-69.8HRCT-ND
- SW1: DIGIKEY https://www.digikey.de/en/products/detail/e-switch/TL3305AF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 -> EG5353CT-ND
- U2: DIGIKEY https://www.ebay.de/itm/152524560455?hash=item23832c1847:g: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 -> 1428-1007-1-ND
- U3: DIGIKEY https://www.digikey.de/en/products/detail/stmicroelectronic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 -> 497-11518-ND
- Y1: DIGIKEY https://www.digikey.de/en/products/detail/abracon-llc/ABLS-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 -> 535-14944-1-ND

Commit message: 
Connections:
- net GPS_IRQ: no longer names the net of U3.39 (PB3)
Other:
- sheet GPS ports: added none; removed EXTINT
Changed lines of the file:
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@@
-    )
-  )
-  (global_label "GPS_IRQ" (shape output) (at 189.865 156.845 180) (fields_autoplaced)
-    (effects (font (size 1.27 1.27)) (justify right))
-    (property "Intersheet References" "${INTERSHEET_REFS}" (id 0) (at 179.5295 156.7656 0)
-      (effects (font (size 1.27 1.27)) (justify right) hide)
     )
   )
@@
     (effects (font (size 1.27 1.27)) (justify right))
     (property "Intersheet References" "${INTERSHEET_REFS}" (id 0) (at 124.3752 72.3106 0)
-      (effects (font (size 1.27 1.27)) (justify right) hide)
-    )
-  )
-  (global_label "GPS_IRQ" (shape input) (at 136.525 74.93 180) (fields_autoplaced)
-    (effects (font (size 1.27 1.27)) (justify right))
-    (property "Intersheet References" "${INTERSHEET_REFS}" (id 0) (at 126.1895 74.8506 0)
       (effects (font (size 1.27 1.27)) (justify right) hide)
     )
@@
       (effects (font (size 1.27 1.27)) (justify left top))
     )
-    (pin "EXTINT" output (at 189.865 156.845 180)
-      (effects (font (size 1.27 1.27)) (justify left))
-    )
     (pin "MOSI" input (at 189.865 147.955 180)

Commit message: 
Parts:
- U1: DIGIKEY - -> 31-AZ1117CH2-3.3TRG1CT-ND
Changed lines of the file:
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@@
       (effects (font (size 1.27 1.27)) hide)
     )
-    (property "DIGIKEY" "-" (id 4) (at 60.96 20.955 0)
+    (property "DIGIKEY" "31-AZ1117CH2-3.3TRG1CT-ND" (id 4) (at 60.96 20.955 0)
       (effects (font (size 1.27 1.27)) hide)
     )

Commit message: 
Parts:
- C14: footprint Capacitor_SMD:CP_Elec_5x5.9 -> Capacitor_SMD:CP_Elec_5x5.4
Changed lines of the file:
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@@
       (effects (font (size 1.27 1.27)) (justify left))
     )
-    (property "Footprint" "Capacitor_SMD:CP_Elec_5x5.9" (id 2) (at 228.2952 31.115 0)
+    (property "Footprint" "Capacitor_SMD:CP_Elec_5x5.4" (id 2) (at 228.2952 31.115 0)
       (effects (font (size 1.27 1.27)) hide)
     )
@@
     )
     (path "/aa122ab8-03e5-4c5e-a007-ec3e3f5864b8"
-      (reference "C14") (unit 1) (value "10uF") (footprint "Capacitor_SMD:CP_Elec_5x5.9")
+      (reference "C14") (unit 1) (value "10uF") (footprint "Capacitor_SMD:CP_Elec_5x5.4")
     )
     (path "/431ea231-a812-4481-addf-46e53a5f0cb7"
