File: pcb/heli/gps.kicad_sch (KiCad schematic)
At the start: 7 parts, among them J3 CONMHF4-SMD-G-T, U4 NEO-M9N-00B

Commit message: 
Connections:
- net EXTINT: no longer names the net of U4.4 (EXTINT)
Changed lines of the file:
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@@
-    (stroke (width 0) (type default) (color 0 0 0 0))
-  )
-  (wire (pts (xy 119.38 76.2) (xy 121.92 76.2))
     (stroke (width 0) (type default) (color 0 0 0 0))
   )
@@
     (effects (font (size 1.27 1.27)) (justify right))
   )
-  (hierarchical_label "EXTINT" (shape output) (at 119.38 76.2 180)
-    (effects (font (size 1.27 1.27)) (justify right))
-  )

Commit message: 
Parts:
- C28: DIGIKEY 1276-1935-1-ND -> -
Changed lines of the file:
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@@
       (effects (font (size 1.27 1.27)) hide)
     )
-    (property "DIGIKEY" "1276-1935-1-ND" (id 4) (at 208.28 53.34 0)
+    (property "DIGIKEY" "-" (id 4) (at 208.28 53.34 0)
       (effects (font (size 1.27 1.27)) hide)
     )

Commit message: 
Parts:
- U4: footprint ICs:XCVR_NEO-M9N-00B -> lib:XCVR_NEO-M9N-00B
Changed lines of the file:
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@@
     (property "Reference" "U4" (id 0) (at 149.86 47.1002 0))
     (property "Value" "NEO-M9N-00B" (id 1) (at 149.86 49.6371 0))
-    (property "Footprint" "ICs:XCVR_NEO-M9N-00B" (id 2) (at 149.86 78.74 0)
+    (property "Footprint" "lib:XCVR_NEO-M9N-00B" (id 2) (at 149.86 78.74 0)
       (effects (font (size 1.27 1.27)) (justify bottom) hide)
     )

Commit message: 
Parts:
- J3: DIGIKEY 2057-PH1-10-UA-ND -> 343-CONMHF4-SMD-G-TCT-ND
Connections:
- net GPS50ohms: now reaches J3.1, U4.11 (RF_IN)
Changed lines of the file:
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@@
     (stroke (width 0) (type default) (color 0 0 0 0))
+  )
+  (label "GPS50ohms" (at 109.855 66.04 0)
+    (effects (font (size 1.27 1.27)) (justify left bottom))
   )
   (global_label "3.3V" (shape input) (at 190.5 53.34 0) (fields_autoplaced)
@@
       (effects (font (size 1.27 1.27)) (justify bottom) hide)
     )
-    (property "DIGIKEY" "2057-PH1-10-UA-ND" (id 8) (at 105.41 66.04 0)
+    (property "DIGIKEY" "343-CONMHF4-SMD-G-TCT-ND" (id 8) (at 105.41 66.04 0)
       (effects (font (size 1.27 1.27)) hide)
     )
